File: ID_EEPROM.kicad_sch (KiCad schematic)
At the start: 2 parts, among them U2 M24C64

Commit message: PCB design
In progress
Other:
- title: MMS3 Hat template small (Change Me) -> MMS3 Hat servo controller
Changed lines of the file:
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@@
 	(paper "A4")
 	(title_block
-		(title "MMS3 Hat template small (Change Me)")
+		(title "MMS3 Hat servo controller")
 		(date "2026-02-25")
 		(rev "A")
