File: Power_Connector.kicad_sch (KiCad schematic)
At the start: 3 parts, among them J4 AMASS XT60 Male, J5 AMASS XT60 Female

Commit message: polished the schemtic
Parts:
- removed D3: SS510C, SS510C:SMC_L7.1-W6.2-LS8.1-RD, symbol SS510C:SS510C
- added D4: SS510C, SS510C:SMC_L7.1-W6.2-LS8.1-RD, symbol SS510C:SS510C
Connections:
- net Vin renamed VIN_BRD
- net VIN_BRD: now also D4.2 (A)
- new net VIN_Chainbus: D4.1 (K)
Other:
- note removed: "If you remove this, add direct connection betwen Vin and BRD_VIN"

Commit message: PCB design
In progress
Other:
- title: MMS3 Hat template small (Change Me) -> MMS3 Hat servo controller
Changed lines of the file:
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@@
 	(paper "A4")
 	(title_block
-		(title "MMS3 Hat template small (Change Me)")
+		(title "MMS3 Hat servo controller")
 		(date "2026-02-25")
 		(rev "A")

Commit message: Revieved by Wojtek
Parts:
- removed D4: SS510C, SS510C:SMC_L7.1-W6.2-LS8.1-RD, symbol SS510C:SS510C
- added D1: M7, PCM_JLCPCB:D_SMA, symbol PCM_JLCPCB-Diodes:General,M7
Connections:
- net VIN_BRD: now also D1.2
- net VIN_Chainbus: now also D1.1
Changed lines of the file:
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@@
+	(wire
+		(pts
+			(xy 147.32 101.6) (xy 152.4 101.6)
+		)
+		(stroke
+			(width 0)
+			(type default)
+		)
+	)
 	(wire
 		(pts
@@
 		(pts
 			(xy 121.92 110.49) (xy 128.27 110.49)
-		)
-		(stroke
-			(width 0)
-			(type default)
-		)
-	)
-	(wire
-		(pts
-			(xy 149.86 101.6) (xy 152.4 101.6)
 		)
 		(stroke
@@
 			(justify left bottom)
 		)
-		(property "Net Class" "50V "
+		(property "Net Class" "50V"
 			(at 126.746 97.282 0)
 			(show_name no)
@@
 			(justify left bottom)
 		)
-		(property "Net Class" "50V "
+		(property "Net Class" "50V"
 			(at 150.876 96.012 0)
 			(show_name no)
@@
 				)
 				(justify right)
-			)
-		)
-	)
-	(symbol
-		(lib_id "SS510C:SS510C")
-		(at 144.78 101.6 180)
-		(unit 1)
-		(body_style 1)
-		(exclude_from_sim no)
-		(in_bom yes)
-		(on_board yes)
-		(in_pos_files yes)
-		(dnp no)
-		(fields_autoplaced yes)
-		(property "Reference" "D4"
-			(at 145.16 95.25 0)
-			(show_name no)
-			(do_not_autoplace no)
-			(effects
-				(font
-					(size 1.27 1.27)
-				)
-			)
-		)
-		(property "Value" "SS510C"
-			(at 145.16 97.79 0)
-			(show_name no)
-			(do_not_autoplace no)
-			(effects
-				(font
-					(size 1.27 1.27)
-				)
-			)
-		)
-		(property "Footprint" "SS510C:SMC_L7.1-W6.2-LS8.1-RD"
-			(at 144.78 93.98 0)
-			(hide yes)
-			(show_name no)
-			(do_not_autoplace no)
-			(effects
-				(font
-					(size 1.27 1.27)
-				)
-			)
-		)
-		(property "Datasheet" "https://lcsc.com/product-detail/Schottky-Barrier-Diodes-SBD_SS510C_C123944.html"
-			(at 144.78 91.44 0)
-			(hide yes)
-			(show_name no)
-			(do_not_autoplace no)
-			(effects
-				(font
-					(size 1.27 1.27)
-				)
-			)
-		)
-		(property "Description" ""
-			(at 144.78 101.6 0)
-			(hide yes)
-			(show_name no)
-			(do_not_autoplace no)
-			(effects
-				(font
-					(size 1.27 1.27)
-				)
-			)
-		)
-		(property "Manufacturer" "晶导微电子"
-			(at 144.78 88.9 0)
-			(hide yes)
-			(show_name no)
-			(do_not_autoplace no)
-			(effects
-				(font
-					(size 1.27 1.27)
-				)
-			)
-		)
-		(property "MPN" "SS510C"
-			(at 144.78 86.36 0)
-			(hide yes)
-			(show_name no)
-			(do_not_autoplace no)
-			(effects
-				(font
-					(size 1.27 1.27)
-				)
-			)
-		)
-		(property "LCSC Part" "C123944"
-			(at 144.78 83.82 0)
-			(hide yes)
-			(show_name no)
-			(do_not_autoplace no)
-			(effects
-				(font
-					(size 1.27 1.27)
-				)
-			)
-		)
-		(pin "2"
-		)
-		(pin "1"
-		)
-		(instances
-			(project "MMS3_hat_templates"
-				(path "/6596548a-44e0-46d8-8624-fd71cf4a3e17/99cf0a47-7576-4da2-b5b4-2714d9e150a8"
-					(reference "D4")
-					(unit 1)
-				)
 			)
 		)
@@
 		)
 		(instances
-			(project "MMS3_hat_templates"
+			(project "MMS3_hat_servo"
 				(path "/6596548a-44e0-46d8-8624-fd71cf4a3e17/99cf0a47-7576-4da2-b5b4-2714d9e150a8"
 					(reference "J5")
@@
 		)
 		(instances
-			(project "MMS3_hat_templates"
+			(project "MMS3_hat_servo"
 				(path "/6596548a-44e0-46d8-8624-fd71cf4a3e17/99cf0a47-7576-4da2-b5b4-2714d9e150a8"
 					(reference "#PWR040")
@@
 		)
 		(instances
-			(project "MMS3_hat_templates"
+			(project "MMS3_hat_servo"
 				(path "/6596548a-44e0-46d8-8624-fd71cf4a3e17/99cf0a47-7576-4da2-b5b4-2714d9e150a8"
 					(reference "#FLG03")
@@
 		)
 		(instances
-			(project "MMS3_hat_templates"
+			(project "MMS3_hat_servo"
 				(path "/6596548a-44e0-46d8-8624-fd71cf4a3e17/99cf0a47-7576-4da2-b5b4-2714d9e150a8"
 					(reference "J4")
@@
 		)
 		(instances
-			(project "MMS3_hat_templates"
+			(project "MMS3_hat_servo"
 				(path "/6596548a-44e0-46d8-8624-fd71cf4a3e17/99cf0a47-7576-4da2-b5b4-2714d9e150a8"
 					(reference "#FLG02")
 					(unit 1)
 				)
+			)
+		)
+	)
+	(symbol
+		(lib_id "PCM_JLCPCB-Diodes:General,M7")
+		(at 143.51 101.6 90)
+		(unit 1)
+		(body_style 1)
+		(exclude_from_sim no)
+		(in_bom yes)
+		(on_board yes)
+		(in_pos_files yes)
+		(dnp no)
+		(fields_autoplaced yes)
+		(property "Reference" "D1"
+			(at 143.51 95.25 90)
+			(show_name no)
+			(do_not_autoplace no)
+			(effects
+				(font
+					(size 1.27 1.27)
+				)
+			)
+		)
+		(property "Value" "M7"
+			(at 143.51 97.79 90)
+			(show_name no)
+			(do_not_autoplace no)
+			(effects
+				(font
+					(size 0.8 0.8)
+				)
+			)
+		)
+		(property "Footprint" "PCM_JLCPCB:D_SMA"
+			(at 143.51 103.378 90)
+			(hide yes)
+			(show_name no)
+			(do_not_autoplace no)
+			(effects
+				(font
+					(size 1.27 1.27)
+				)
+			)
+		)
+		(property "Datasheet" "https://www.lcsc.com/datasheet/lcsc_datasheet_2407101107_MDD-Microdiode-Semiconductor-M7_C95872.pdf"
+			(at 143.51 101.6 0)
+			(hide yes)
+			(show_name no)
+			(do_not_autoplace no)
+			(effects
+				(font
+					(size 1.27 1.27)
+				)
+			)
+		)
+		(property "Description" "1A Independent Type 1kV 1.1V@1A SMA(DO-214AC) Diodes - General Purpose ROHS"
+			(at 143.51 101.6 0)
+			(hide yes)
+			(show_name no)
+			(do_not_autoplace no)
+			(effects
+				(font
+					(size 1.27 1.27)
+				)
+			)
+		)
+		(property "LCSC" "C95872"
+			(at 143.51 101.6 0)
+			(hide yes)
+			(show_name no)
+			(do_not_autoplace no)
+			(effects
+				(font
+					(size 1.27 1.27)
+				)
+			)
+		)
+		(property "Stock" "3256855"
+			(at 143.51 101.6 0)
+			(hide yes)
+			(show_name no)
+			(do_not_autoplace no)
+			(effects
+				(font
+					(size 1.27 1.27)
+				)
+			)
+		)
+		(property "Price" "0.011USD"
+			(at 143.51 101.6 0)
+			(hide yes)
+			(show_name no)
+			(do_not_autoplace no)
+			(effects
+				(font
+					(size 1.27 1.27)
+				)
+			)
+		)
+		(property "Process" "SMT"
+			(at 143.51 101.6 0)
+			(hide yes)
+			(show_name no)
+			(do_not_autoplace no)
+			(effects
+				(font
+					(size 1.27 1.27)
+				)
+			)
+		)
+		(property "Minimum Qty" "5"
+			(at 143.51 101.6 0)
+			(hide yes)
+			(show_name no)
+			(do_not_autoplace no)
+			(effects
+				(font
+					(size 1.27 1.27)
+				)
+			)
+		)
+		(property "Attrition Qty" "10"
+			(at 143.51 101.6 0)
+			(hide yes)
+			(show_name no)
+			(do_not_autoplace no)
+			(effects
+				(font
+					(size 1.27 1.27)
+				)
+			)
+		)
+		(property "Class" "Basic Component"
+			(at 143.51 101.6 0)
+			(hide yes)
+			(show_name no)
+			(do_not_autoplace no)
+			(effects
+				(font
+					(size 1.27 1.27)
+				)
+			)
+		)
+		(property "Category" "Diodes,Diodes - General Purpose"
+			(at 143.51 101.6 0)
+			(hide yes)
+			(show_name no)
+			(do_not_autoplace no)
+			(effects
+				(font
+					(size 1.27 1.27)
+				)
+			)
+		)
+		(property "Manufacturer" "MDD（Microdiode Electronics）"
+			(at 143.51 101.6 0)
+			(hide yes)
+			(show_name no)
+			(do_not_autoplace no)
+			(effects
+				(font
+					(size 1.27 1.27)
+				)
+			)
+		)
+		(property "Part" "M7"
+			(at 143.51 101.6 0)
+			(hide yes)
+			(show_name no)
+			(do_not_autoplace no)
+			(effects
+				(font
+					(size 1.27 1.27)
+				)
+			)
+		)
+		(property "Rectified Current" "1A"
+			(at 143.51 101.6 0)
+			(hide yes)
+			(show_name no)
+			(do_not_autoplace no)
+			(effects
+				(font
+					(size 1.27 1.27)
+				)
+			)
+		)
+		(property "Forward Voltage (Vf@If)" "1.1V@1A"
+			(at 143.51 101.6 0)
+			(hide yes)
+			(show_name no)
+			(do_not_autoplace no)
+			(effects
+				(font
+					(size 1.27 1.27)
+				)
+			)
+		)
+		(property "Reverse Voltage (Vr)" "1kV"
+			(at 143.51 101.6 0)
+			(hide yes)
+			(show_name no)
+			(do_not_autoplace no)
+			(effects
+				(font
+					(size 1.27 1.27)
+				)
+			)
+		)
+		(property "Diode Configuration" "Independent Type"
+			(at 143.51 101.6 0)
+			(hide yes)
+			(show_name no)
+			(do_not_autoplace no)
+			(effects
+				(font
+					(size 1.27 1.27)
+				)
+			)
+		)
+		(property "Reverse Leakage Current" "5uA@1kV"
+			(at 143.51 101.6 0)
+			(hide yes)
+			(show_name no)
+			(do_not_autoplace no)
+			(effects
+				(font
+					(size 1.27 1.27)
+				)
+			)
+		)
+		(pin "1"
+		)
+		(pin "2"
+		)
+		(instances
+			(project "MMS3_hat_servo"
+				(path "/6596548a-44e0-46d8-8624-fd71cf4a3e17/99cf0a47-7576-4da2-b5b4-2714d9e150a8"
+					(reference "D1")
+					(unit 1)
+				)
