File: Hardware/MMS3_hat_servo.kicad_pcb (KiCad board)
At the start: 2 copper layers, 100 x 50 mm, 59 parts, among them J1 Chainbus in, J10 Conn_01x03, J2 Chainbus Out, J3 Conn_01x04_Pin, J4 AMASS XT60 Male, J5 AMASS XT60 Female, J7 Conn_01x03, J8 Conn_01x03, J9 Conn_01x03, Q4 AO3400A, Q5 AO3400A, U1 PCA9685PW,118, U2 M24C64, U3 SN74CB3Q3245PWR, U4 AMS1117

Commit message: added documentation
Parts:
- moved C30 0.11 mm to (149.5, 108.5)
Routing:
- net /Bus_switch/Chainbus.SDA: track 72.3 -> 73.3 mm

Commit message: generated gerber
Other:
- board text added: "MMS3 Hat servo controller version 1.0 by Szymon Filip"
- board text removed: "Hat servo controller version 1.0 by Szymon Filip"
Changed lines of the file:
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@@
 	(paper "A4")
 	(title_block
-		(title "MMS3 Hat Stepper Controler")
+		(title "MMS3 Hat Servo Controller")
 		(date "2026-02-25")
-		(rev "R0")
-		(comment 1 "Made by Wojciech Szafrański")
+		(rev "V1.0")
+		(comment 1 "Made by Szymon FIlip")
 		(comment 2 "Designed in poland")
 		(comment 3 "MMS3 Hat based on Chainbus")
@@
 		)
 	)
+	(gr_text "MMS3 Hat\nservo controller \nversion 1.0 \nby Szymon Filip"
+		(at 94.2 117.4 0)
+		(layer "F.SilkS")
+		(effects
+			(font
+				(size 2 2)
+			)
+			(justify bottom)
+		)
+	)
 	(gr_text "This is prototype device\nIt is not certified according\nto current EU laws.\nDo not sell or use outside of\nresearch purposes."
 		(at 137.2 109.65 0)
@@
 		)
 	)
-	(gr_text "Hat servo controller \nversion 1.0 \nby Szymon Filip"
-		(at 94.75 113.25 0)
-		(layer "B.SilkS")
-		(effects
-			(font
-				(size 1 1)
-				(thickness 0.1)
-			)
-			(justify bottom mirror)
-		)
-	)
